File: F0DisplayBoard/F0DisplayBoard.sch (KiCad schematic (older format))
At the start: 36 parts, among them J1 NHD-C0216CZ-FSW-FBW-3V3, J2 USB_B_Micro, U1 STM32F051R8T6TR, U2 ROTARY_ENC_PEC12R, U3 AZ1117EH-3.3TRG1, U4 FT232RLREEL, X1 ABLS7M2_16MHz_XTAL

Commit message: sch: Removed some connectors to make room on board. pcb: rough routing, difficulty with traces cutting into planes. May restart routing of most signals
Parts:
- added D1, D2, D3, D4, D5, D6, D7, D8: LED, LED_SMD:LED_0805_2012Metric_Pad1.15x1.40mm_HandSolder, symbol Device:LED
- added J6: CONN_PB, Connector_PinHeader_2.54mm:PinHeader_1x16_P2.54mm_Vertical, symbol Connector:Conn_01x16_Male
- added J8: CONN_FTDI, Connector_PinHeader_2.54mm:PinHeader_1x05_P2.54mm_Vertical, symbol Connector:Conn_01x05_Male
- added J9: CONN_ROT, Connector_PinHeader_2.54mm:PinHeader_1x03_P2.54mm_Vertical, symbol Connector:Conn_01x03_Male
- added R10, R11, R12, R13, R14, R15, R16, R17, R6, R7, R8, R9: 1K, Resistor_SMD:R_0805_2012Metric_Pad1.15x1.40mm_HandSolder, symbol Device:R
- added SW2, SW3, SW4, SW5: SW_Push, TACTILE_SW:PTS645SK43SMTR92LFS, symbol TACTILE_SW:SW_Push
- C1: renamed from C3; footprint (none) -> Capacitor_SMD:C_0805_2012Metric_Pad1.15x1.40mm_HandSolder
- C10: renamed from C2; footprint (none) -> Capacitor_SMD:C_0805_2012Metric_Pad1.15x1.40mm_HandSolder
- C11, C12, C13, C14, C15, C16: renamed from C?; footprint (none) -> Capacitor_SMD:C_0805_2012Metric_Pad1.15x1.40mm_HandSolder
- C2: renamed from C4; footprint (none) -> Capacitor_SMD:C_0805_2012Metric_Pad1.15x1.40mm_HandSolder
- C3: renamed from C5; footprint (none) -> Capacitor_SMD:C_0805_2012Metric_Pad1.15x1.40mm_HandSolder
- C4: renamed from C6; footprint (none) -> Capacitor_SMD:C_0805_2012Metric_Pad1.15x1.40mm_HandSolder
- C5: renamed from C7; footprint (none) -> Capacitor_SMD:C_0805_2012Metric_Pad1.15x1.40mm_HandSolder
- C6: renamed from C8; footprint (none) -> Capacitor_SMD:C_0805_2012Metric_Pad1.15x1.40mm_HandSolder
- C7: renamed from C1; footprint (none) -> Capacitor_SMD:C_0805_2012Metric_Pad1.15x1.40mm_HandSolder
- C8: renamed from C9; footprint (none) -> Capacitor_SMD:C_0805_2012Metric_Pad1.15x1.40mm_HandSolder
- C9: renamed from C10; footprint (none) -> Capacitor_SMD:C_0805_2012Metric_Pad1.15x1.40mm_HandSolder
- J1: renamed from J2; footprint (none) -> MICROUSB:CUIDEVICES_UJ2-MIBH-4-SMT-TR
- J10: renamed from J?; footprint (none) -> Connector_PinHeader_2.54mm:PinHeader_1x03_P2.54mm_Vertical
- J2, J3: renamed from J?; footprint (none) -> Connector_PinHeader_2.54mm:PinHeader_1x02_P2.54mm_Vertical
- J7: renamed from J?; value Conn_01x08_Male -> CONN_DEBUG; footprint (none) -> Connector_PinHeader_2.54mm:PinHeader_1x08_P2.54mm_Vertical
- JP1, JP2: renamed from JP?; footprint (none) -> Connector_PinHeader_2.54mm:PinHeader_1x03_P2.54mm_Vertical
- R1: renamed from R2; footprint (none) -> Resistor_SMD:R_0805_2012Metric_Pad1.15x1.40mm_HandSolder
- R3, R4, R5: renamed from R?; footprint (none) -> Resistor_SMD:R_0805_2012Metric_Pad1.15x1.40mm_HandSolder
- SW1: renamed from SW?; footprint (none) -> TACTILE_SW:PTS645SK43SMTR92LFS; symbol Switch:SW_Push -> TACTILE_SW:SW_Push
- renumbered J1 to J5, R1 to R2, U3 to U1, U4 to U2, U2 to U3, U1 to U4
Connections:
- net +3V3: now also R1.1, R17.1, R6.1, R7.1, R8.1
- net +5V: no longer R1.1
- net DISP_CSB: now also J6.6 (Pin_6)
- net DISP_RS: now also J6.10 (Pin_10)
- net DISP_RST: now also J6.9 (Pin_9)
- net DISP_SCL: now also J6.7 (Pin_7)
- net DISP_SI: now also J6.8 (Pin_8)
- net FT_CTS: now also J8.2 (Pin_2)
- net FT_PWREN: now also J8.5 (Pin_5)
- net FT_RTS: now also J8.1 (Pin_1)
- net FT_RX: now also J8.3 (Pin_3)
- net FT_TX: now also J8.4 (Pin_4)
- net GND: now also SW1.2, D1.1 (K), D2.1 (K), D3.1 (K), D4.1 (K), D5.1 (K), D6.1 (K), D7.1 (K), D8.1 (K), SW2.3, SW2.4, SW3.3, SW3.4, SW4.3, SW4.4, SW5.3, SW5.4
- net NRST: now also SW1.3, SW1.4; no longer SW1.2
- net ROT_CHA: now also J9.2 (Pin_2)
- net ROT_CHB: now also J9.3 (Pin_3)
- net ROT_SW1: now also J6.16 (Pin_16), J9.1 (Pin_1)
- net VCAP2: now reaches C12.2, U4.125 (VCAP_2)
- net VBAT: now reaches C13.2, U4.6 (VBAT)
- net VCAP1: now reaches C11.1, U4.81 (VCAP_1)
- net PC15: now reaches U4.10 (PC15-OSC32_OUT(PC15))
- net PD12: now reaches U4.100 (PD12)
- net PD13: now reaches U4.101 (PD13)
- net PD14: now reaches U4.104 (PD14)
- net PD15: now reaches U4.105 (PD15)
- net PC6: now reaches U4.115 (PC6)
- net PC6: now also R11.2
- net PC7: now reaches U4.116 (PC7)
- net PC7: now also R12.2
- net PC8: now reaches U4.117 (PC8)
- net PC8: now also R13.2
- net PC9: now reaches U4.118 (PC9)
- net PC9: now also R14.2
- net PA11: now reaches U4.122 (PA11)
- net PA12: now reaches U4.123 (PA12)
- net JTMS-SWDIO: now reaches J7.4 (Pin_4), U4.124 (PA13(JTMS-SWDIO))
- net JTCK-SWCLK: now reaches J7.2 (Pin_2), U4.137 (PA14(JTCK-SWCLK))
- net JTDI: now reaches J7.7 (Pin_7), U4.138 (PA15(JTDI))
- net PC10: now reaches U4.139 (PC10)
- net PC10: now also R15.2
- net PC11: now reaches U4.140 (PC11)
- net PC11: now also R16.2
- net PC12: now reaches U4.141 (PC12)
- net PD0: now reaches U4.142 (PD0)
- net PD1: now reaches U4.143 (PD1)
- net PD2: now reaches U4.144 (PD2)
- net PD3: now reaches U4.145 (PD3)
- net PD4: now reaches U4.146 (PD4)
- net PD5: now reaches U4.147 (PD5)
- net PD6: now reaches U4.150 (PD6)
- net PD7: now reaches U4.151 (PD7)
- net JTDO: now reaches J7.6 (Pin_6), U4.161 (PB3(JTDO/TRACESWO))
- net JTDO: now also J6.4 (Pin_4)
- net NJTRST: now reaches J7.5 (Pin_5), U4.162 (PB4(NJTRST))
- net NJTRST: now also J6.5 (Pin_5)
- net PC0: now reaches U4.32 (PC0)
- net PC0: now also R6.2, SW2.1, SW2.2
- net PC1: now reaches U4.33 (PC1)
- net PC1: now also R7.2, SW3.1, SW3.2
- net PC2: now reaches U4.34 (PC2)
- net PC2: now also R8.2, SW4.1, SW4.2
- net PC3: now reaches U4.35 (PC3)
- net PC3: now also R17.2, SW5.1, SW5.2
- net PA4: now reaches U4.50 (PA4)
- net PA5: now reaches U4.51 (PA5)
- net PA6: now reaches U4.52 (PA6)
- net PA7: now reaches U4.53 (PA7)
- net PC4: now reaches U4.54 (PC4)
- net PC4: now also R9.2
- net PC5: now reaches U4.55 (PC5)
- net PC5: now also R10.2
- net PB0: now reaches U4.56 (PB0)
- net PB0: now also J6.1 (Pin_1)
- net PB1: now reaches U4.57 (PB1)
- net PB1: now also J6.2 (Pin_2)
- net BOOT1: now reaches U4.58 (PB2-BOOT1(PB2))
- net BOOT1: now also J6.3 (Pin_3)
- net PB10: now reaches U4.79 (PB10)
- net PB10: now also J6.11 (Pin_11)
- net PC13: now reaches U4.8 (PC13)
- net PB11: now reaches U4.80 (PB11)
- net PB11: now also J6.12 (Pin_12)
- net PC14: now reaches U4.9 (PC14-OSC32_IN(PC14))
- net PB12: now reaches U4.92 (PB12)
- net PB12: now also J6.13 (Pin_13)
- net PB13: now reaches U4.93 (PB13)
- net PB13: now also J6.14 (Pin_14)
- net PB14: now reaches U4.94 (PB14)
- net PB14: now also J6.15 (Pin_15)
- net PD8: now reaches U4.96 (PD8)
- net PD9: now reaches U4.97 (PD9)
- net PD10: now reaches U4.98 (PD10)
- net PD11: now reaches U4.99 (PD11)
- net VBUS: now reaches C3.1, FB1.2, J1.1 (VBUS)
- net D-: now reaches J1.2 (D-), U2.16 (USBDM)
- net D+: now reaches J1.3 (D+), U2.15 (USBDP)
- net FT_3V3OUT: now reaches C5.1, U2.17 (3V3OUT)
- new net: D1.2 (A), R9.1
- new net: D2.2 (A), R10.1
- new net: D3.2 (A), R11.1
- new net: D4.2 (A), R12.1
- new net: D5.2 (A), R13.1
- new net: D6.2 (A), R14.1
- new net: D7.2 (A), R15.1
- new net: D8.2 (A), R16.1
- no-connect marks 11 -> 85
Other:
- note added: "STM32 IO Breakouts"
- note added: "Test Buttons"
- note added: "Test LEDs"
- note removed: "TODO:\n -Make sure regulator/usb stuff is OK\n -Add Test Points / Test Jumpers\n -Extra Buttons / LEDs?"
- moved on the sheet: C1, C10, C11, C12, C13, C14, C15, C16, C2, C3, C4, C5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

Commit message: Rev2 completed   -Added current-limiting resitstor for LCD backlight   -Fixed microcontroller footprint   -Board size reduced
Parts:
- removed C16: 1uF, Capacitor_SMD:C_0805_2012Metric_Pad1.15x1.40mm_HandSolder, symbol Device:C
- removed J10: CONN_STMPWR, Connector_PinHeader_2.54mm:PinHeader_1x03_P2.54mm_Vertical, symbol Connector:Conn_01x03_Male
- removed U4: STM32F051R8T6TR, STM32F051R8T6:QFP50P2600X2600X160-176N, symbol STM32F0:STM32F051R8T6TR
- added IC1: STM32F051R8T6TR, LibraryLoader:QFP50P1200X1200X160-64N, symbol LibraryLoader:STM32F051R8T6TR
- added JP3: JUMPER_BOOT0, Connector_PinHeader_2.54mm:PinHeader_1x02_P2.54mm_Vertical, symbol Device:Jumper_NO_Small
- C13: value 100nF -> 4.7uF
- C14: value 4.7uF -> 10nF
- C15: value 10nF -> 1uF
- R3: value 10K -> 1K
Connections:
- net +3.3VA is gone; now on net +3V3: C15.1
- net VCAP1 is gone; now on net VBAT: C11.1
- net VCAP2 is gone; now on net GND: C12.2
- net +3V3: now also C11.2, C12.1, IC1.13 (VDDA), IC1.32 (VDD_1), IC1.64 (VDD_2), JP3.2
- net BOOT0: now also R4.1, IC1.60 (BOOT0), JP3.1; no longer R4.2
- net BOOT1: now also IC1.28 (PB2)
- net DISP_CSB: now also IC1.57 (PB5)
- net DISP_RS: now also IC1.62 (PB9)
- net DISP_RST: now also IC1.61 (PB8)
- net DISP_SCL: now also IC1.58 (PB6)
- net DISP_SI: now also IC1.59 (PB7)
- net FT_CTS: now also IC1.15 (PA1)
- net FT_PWREN: now also IC1.43 (PA10)
- net FT_RTS: now also IC1.14 (PA0)
- net FT_RX: now also IC1.16 (PA2)
- net FT_TX: now also IC1.17 (PA3)
- net GND: now also C13.2, R4.2, IC1.12 (VSSA), IC1.31 (VSS_1), IC1.63 (VSS_2); no longer C11.2, C12.1, J5.K (LED-), R4.1
- net JTCK-SWCLK: now also IC1.49 (PA14)
- net JTDI: now also IC1.50 (PA15)
- net JTDO: now also IC1.55 (PB3)
- net JTMS-SWDIO: now also IC1.46 (PA13)
- net NJTRST: now also IC1.56 (PB4)
- net NRST: now also IC1.7 (NRST)
- net PB0: now also IC1.26 (PB0)
- net PB1: now also IC1.27 (PB1)
- net PB10: now also IC1.29 (PB10)
- net PB11: now also IC1.30 (PB11)
- net PB12: now also IC1.33 (PB12)
- net PB13: now also IC1.34 (PB13)
- net PB14: now also IC1.35 (PB14)
- net PC0: now also IC1.8 (PC0)
- net PC1: now also IC1.9 (PC1)
- net PC10: now also IC1.51 (PC10)
- net PC11: now also IC1.52 (PC11)
- net PC2: now also IC1.10 (PC2)
- net PC3: now also IC1.11 (PC3)
- net PC4: now also IC1.24 (PC4)
- net PC5: now also IC1.25 (PC5)
- net PC6: now also IC1.37 (PC6)
- net PC7: now also IC1.38 (PC7)
- net PC8: now also IC1.39 (PC8)
- net PC9: now also IC1.40 (PC9)
- net ROT_CHA: now also IC1.41 (PA8)
- net ROT_CHB: now also IC1.42 (PA9)
- net ROT_SW1: now also IC1.36 (PB15)
- net VBAT: now also IC1.1 (VBAT); no longer C13.2
- net XTAL1: now also IC1.5 (PF0-OSC_IN)
- net XTAL2: now also IC1.6 (PF1-OSC_OUT)
- net BYPASS_REG renamed DISP_LED-
- net DISP_LED-: now also J5.K (LED-)
- no-connect marks 85 -> 26
Other:
- note removed: "STM32 Power Connections"
- note removed: "Test Connector\n"
- moved on the sheet: C10, C7, C8, C9, D1, D2, D3, D4, D5, D6, D7, D8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
